File: Preamp.kicad_pcb (KiCad board)
At the start: 2 copper layers, 285 x 74 mm, 183 parts, among them J1 Conn_01x03, J10 RCAJack, J11 XLR4BODYPIN, J12 XLR4BODYPIN, J13 XLR4BODYPIN, J14 RCAJack, J15 RCAJack, J16 XLR4BODYPIN, J17 XLR4BODYPIN, J18 RCAJack, J19 RCAJack, J2 Conn_01x02, J20 RCAJack, J21 RCAJack, J22 Jack-DC, J23 Conn_01x02, J24 Conn_01x02, J25 Conn_01x01, J26 Conn_01x01, J27 Conn_01x01, J28 Conn_01x01, J3 Conn_01x02, J4 RCAJack, J5 RCAJack, J6 Conn_01x01, J7 Conn_01x01, J8 Conn_01x01, J9 Conn_01x01, SW1 SW_SPST, SW2 SW_SPST, SW3 SW_SPST, U1 LM317, U10 THAT1200, U11 THAT1200, U2 LM337, U3 LM4562, U4 LM4562, U5 LM4562, U6 LM4562, U7 THAT1646, U8 THAT1646, U9 THAT1646

Commit message: remove screwy UVLO
Parts:
- added C58: 10 uF, Capacitors_THT:CP_Radial_D5.0mm_P2.50mm, F.Cu at (99.7, 101.4)
- added D17: 1N4739A, Diodes_THT:D_DO-41_SOD81_P7.62mm_Horizontal, F.Cu at (89.4, 95.3)
- added D18: 1N4007, Diodes_THT:D_DO-41_SOD81_P7.62mm_Horizontal, F.Cu at (107.5, 95.5)
- added Q1: 2N3904, TO_SOT_Packages_THT:TO-92_Inline_Wide, F.Cu at (92.0, 91.8)
- added R41: 10k, Resistors_THT:R_Axial_DIN0207_L6.3mm_D2.5mm_P7.62mm_Horizontal, F.Cu at (89.2, 99.2)
- added R42: 10k, Resistors_THT:R_Axial_DIN0207_L6.3mm_D2.5mm_P7.62mm_Horizontal, F.Cu at (89.2, 102.7)
- added RLY8: DPDTRelay, Preamp:G2VRelay, F.Cu at (101.0, 88.5)
- R23, R43: value 75R -> 4R7
- moved D12 193.0 mm to (89.2, 116.5), turned to 0 degrees
- moved R12 185.6 mm to (96.8, 108.5), turned to 180 degrees
- moved R43 53.4 mm to (114.0, 79.3), turned to 270 degrees
- moved R23 49.2 mm to (110.2, 79.2), turned to 270 degrees
- moved R5 46.3 mm to (82.0, 110.9)
- moved R4 45.4 mm to (83.6, 83.5), turned to 180 degrees
- moved C2 42.3 mm to (77.7, 68.8)
- moved R3 41.4 mm to (85.6, 118.5), turned to 90 degrees
- moved R51 41.4 mm to (145.5, 65.5)
- moved R53 40.4 mm to (80.8, 64.6), turned to 90 degrees
- moved C4 37.6 mm to (83.7, 106.5)
- moved RV4 37.3 mm to (237.9, 118.9)
- moved RV6 37.3 mm to (271.9, 118.9)
- moved C10 37.3 mm to (316.1, 99.6)
- moved C15 37.3 mm to (175.3, 111.5)
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Connections:
- C4 pad 1: +15V -> RECT15P
- C5 pad 2: -15V -> RECT15N
- D16 pad 2: -15V -> RECT15N
- D7 pad 2: +15V -> RECT15P
- D8 pad 1: -15V -> RECT15N
- J23 pad 1: Net-(J22-Pad1) -> Net-(J22-Pad2)
- R12 pad 2: +15V -> RECT15P
- R23 pad 1: -15V -> Net-(R23-Pad1)
- R23 pad 2: GND -> +15V
- R43 pad 1: +15V -> Net-(R43-Pad1)
- R43 pad 2: GND -> -15V
- R5 pad 1: +15V -> RECT15P
- R6 pad 1: -15V -> RECT15N
- RLY7 pad 2: Net-(J22-Pad2) -> Net-(J22-Pad1)
- RLY7 pad 5: -15V -> RECT15N
- SW1 pad 1: +15V -> RECT15P
- SW2 pad 2: +15V -> RECT15P
- SW3 pad 2: -15V -> RECT15N
- U1 pad 2: +15V -> RECT15P
- U2 pad 3: -15V -> RECT15N
Routing:
- net RECT15P: track 0.00 -> 270.4 mm
- net +15V: track 764.6 -> 640.7 mm
- net RECT15N: track 0.00 -> 103.0 mm
- net -15V: track 692.8 -> 614.1 mm, vias 6 -> 7
- net Net-(J22-Pad2): track 36.2 -> 9.07 mm
- net Net-(C58-Pad2): track 0.00 -> 21.6 mm
- net Net-(D17-Pad2): track 0.00 -> 20.5 mm
- net Net-(J22-Pad1): track 21.6 -> 4.56 mm
- net Net-(J3-Pad1): track 110.7 -> 127.1 mm
- net Net-(D11-Pad1): track 109.4 -> 125.7 mm
- net Net-(R23-Pad1): track 0.00 -> 14.7 mm
- net Net-(C1-Pad1): track 56.7 -> 42.1 mm
- net Net-(C55-Pad1): track 44.9 -> 57.3 mm
- net Net-(R43-Pad1): track 0.00 -> 12.1 mm
- net Net-(J19-Pad2): track 26.5 -> 36.4 mm
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Other:
- board size 285 x 74 mm -> 300 x 74 mm
- board text added: "REMOTE OUT"
- board text added: "TONE BYPASS"
- board text removed: "REMOTE OUT POWERED"
- board text removed: "TONE BYPASS SWITCH"
