File: Preamp.kicad_pcb (KiCad board)
At the start: 2 copper layers, 300 x 74 mm, 190 parts, among them J1 Conn_01x03, J10 RCAJack, J11 XLR4BODYPIN, J12 XLR4BODYPIN, J13 XLR4BODYPIN, J14 RCAJack, J15 RCAJack, J16 XLR4BODYPIN, J17 XLR4BODYPIN, J18 RCAJack, J19 RCAJack, J2 Conn_01x02, J20 RCAJack, J21 RCAJack, J22 Jack-DC, J23 Conn_01x02, J24 Conn_01x02, J25 Conn_01x01, J26 Conn_01x01, J27 Conn_01x01, J28 Conn_01x01, J3 Conn_01x02, J4 RCAJack, J5 RCAJack, J6 Conn_01x01, J7 Conn_01x01, J8 Conn_01x01, J9 Conn_01x01, Q1 2N3904, SW1 SW_SPST, SW2 SW_SPST, SW3 SW_SPST, U1 LM317, U10 THAT1200, U11 THAT1200, U2 LM337, U3 LM4562, U4 LM4562, U5 LM4562, U6 LM4562, U7 THAT1646, U8 THAT1646, U9 THAT1646

Commit message: Now grounds all of the outputs when supply is below 20 V
Parts:
- added C59: 100 nF, Capacitors_THT:C_Disc_D5.0mm_W2.5mm_P5.00mm, F.Cu at (103.5, 93.7)
- added C60: 47 uF, Capacitors_THT:CP_Radial_D5.0mm_P2.50mm, F.Cu at (164.6, 89.6)
- added C61: 47 uF, Capacitors_THT:CP_Radial_D5.0mm_P2.50mm, F.Cu at (253.9, 106.0)
- added C62: 47 uF, Capacitors_THT:CP_Radial_D5.0mm_P2.50mm, F.Cu at (258.6, 89.5)
- added Q2: TIP41C, TO_SOT_Packages_THT:TO-220-3_Vertical, F.Cu at (209.2, 62.6)
- added R44: 4R7, Resistors_THT:R_Axial_DIN0309_L9.0mm_D3.2mm_P12.70mm_Horizontal, F.Cu at (103.7, 78.1)
- added RLY10: DPDTRelay, Preamp:G2VRelay, F.Cu at (223.0, 76.7)
- added RLY11: DPDTRelay, Preamp:G2VRelay, F.Cu at (255.3, 82.3)
- added RLY12: DPDTRelay, Preamp:G2VRelay, F.Cu at (295.5, 75.7)
- added RLY9: DPDTRelay, Preamp:G2VRelay, F.Cu at (312.5, 104.6)
- C4, C5: value 47 uF -> 1500 uF; footprint Capacitors_THT:CP_Radial_D7.5mm_P2.50mm -> Capacitors_THT:CP_Radial_D12.5mm_P5.00mm
- C58: value 10 uF -> 100 nF; footprint Capacitors_THT:CP_Radial_D5.0mm_P2.50mm -> Capacitors_THT:C_Disc_D5.0mm_W2.5mm_P5.00mm
- D17: value 1N4739A -> 1N4747A
- Q1: value 2N3904 -> 2N3906
- R23: value 4R7 -> 1k; footprint Resistors_THT:R_Axial_DIN0309_L9.0mm_D3.2mm_P12.70mm_Horizontal -> Resistors_THT:R_Axial_DIN0207_L6.3mm_D2.5mm_P7.62mm_Horizontal
- moved RLY8 218.8 mm to (319.6, 95.3)
- moved Q1 115.0 mm to (205.9, 75.5), turned to 0 degrees
- moved R41 114.2 mm to (200.5, 73.7), turned to 90 degrees
- moved R42 110.6 mm to (193.6, 66.0), turned to 270 degrees
- moved D17 109.9 mm to (197.1, 73.4), turned to 90 degrees
- moved R23 102.3 mm to (212.1, 70.2), turned to 180 degrees
- moved D18 100.3 mm to (201.7, 61.1)
- moved JP1 76.2 mm to (138.7, 53.9)
- moved C46 76.1 mm to (149.8, 69.7)
- moved C43 74.7 mm to (147.6, 54.8)
- moved C47 74.3 mm to (138.4, 61.9)
- moved U10 73.0 mm to (152.7, 65.7)
- moved C44 72.8 mm to (177.3, 59.5), turned to 0 degrees
- moved JP2 64.5 mm to (169.2, 59.7)
- moved C45 63.5 mm to (166.5, 71.9)
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Connections:
- net Net-(D11-Pad1) renamed POWERSW2
- net Net-(J10-Pad2) renamed RIGHTUNBAL
- net Net-(J3-Pad1) renamed POWERSW1
- net Net-(J5-Pad2) renamed LEFTUNBAL
- net Net-(L1-Pad2) renamed SUBPLUS
- net Net-(L2-Pad1) renamed RIGHTPLUS
- net Net-(L3-Pad1) renamed LEFTPLUS
- net Net-(L4-Pad2) renamed SUBMINUS
- net Net-(L5-Pad2) renamed LEFTMINUS
- net Net-(L6-Pad2) renamed RIGHTMINUS
- C4 pad 1: RECT15P -> +15V
- C5 pad 2: RECT15N -> -15V
- C52 pad 2: RIGHTIN -> LEFTIN
- C53 pad 2: LEFTIN -> RIGHTIN
- C58 pad 1: RECT15P -> GND
- D13 pad 1: Net-(D13-Pad1) -> GND
- D13 pad 2: GND -> Net-(D13-Pad2)
- D14 pad 1: Net-(D14-Pad1) -> GND
- D14 pad 2: GND -> Net-(D14-Pad2)
- D16 pad 2: RECT15N -> -15V
- D18 pad 1: RECT15P -> Net-(D18-Pad1)
- D18 pad 2: Net-(C58-Pad2) -> GND
- D7 pad 2: RECT15P -> Net-(C58-Pad2)
- D8 pad 1: RECT15N -> Net-(C59-Pad1)
- J2 pad 1: Net-(D4-Pad2) -> Net-(D1-Pad2)
- J2 pad 2: Net-(D1-Pad2) -> Net-(D4-Pad2)
- J4 pad 2: Net-(J4-Pad2) -> SUBUNBAL
- Q1 pad 1: GND -> +15V
- Q1 pad 2: Net-(D17-Pad2) -> Net-(D17-Pad1)
- Q1 pad 3: Net-(C58-Pad2) -> Net-(Q1-Pad3)
- R12 pad 2: RECT15P -> +15V
- R23 pad 1: Net-(R23-Pad1) -> Net-(Q2-Pad1)
- R23 pad 2: +15V -> Net-(Q1-Pad3)
- R29 pad 1: Net-(J4-Pad2) -> SUBUNBAL
- R31 pad 2: Net-(J4-Pad2) -> SUBUNBAL
- R41 pad 2: RECT15P -> +15V
- R42 pad 1: GND -> -15V
- R43 pad 1: Net-(R43-Pad1) -> +15V
- R43 pad 2: -15V -> Net-(C58-Pad2)
- R5 pad 1: RECT15P -> Net-(C58-Pad2)
- R6 pad 1: RECT15N -> Net-(C59-Pad1)
- RLY3 pad 5: Net-(D13-Pad1) -> Net-(D13-Pad2)
- RLY4 pad 1: Net-(D14-Pad1) -> Net-(D14-Pad2)
- RLY5 pad 5: Net-(D14-Pad1) -> Net-(D14-Pad2)
- RLY6 pad 2: RIGHTIN -> LEFTIN
- RLY6 pad 6: LEFTIN -> RIGHTIN
- RLY7 pad 1: GND -> -15V
- RLY7 pad 2: Net-(J22-Pad1) -> Net-(J24-Pad1)
- RLY7 pad 4: Net-(J23-Pad2) -> Net-(J24-Pad2)
- RLY7 pad 5: RECT15N -> GND
- RLY7 pad 6: Net-(J24-Pad1) -> Net-(J22-Pad1)
- RLY7 pad 8: Net-(J24-Pad2) -> Net-(J23-Pad2)
- RLY8 pad 1: Net-(C58-Pad2) -> GND
- RLY8 pad 2: Net-(R23-Pad1) -> SUBUNBAL
- RLY8 pad 4: RECT15P -> (no net)
- RLY8 pad 5: RECT15P -> Net-(D18-Pad1)
- RLY8 pad 6: Net-(R43-Pad1) -> (no net)
- RLY8 pad 8: RECT15N -> (no net)
- SW1 pad 1: RECT15P -> -15V
- SW1 pad 2: Net-(D13-Pad1) -> Net-(D13-Pad2)
- SW2 pad 1: Net-(D14-Pad1) -> Net-(D14-Pad2)
- SW2 pad 2: RECT15P -> -15V
- SW3 pad 2: RECT15N -> -15V
- U1 pad 2: RECT15P -> Net-(C58-Pad2)
- U2 pad 3: RECT15N -> Net-(C59-Pad1)
Routing:
- net -15V: track 614.1 -> 1149.7 mm, vias 7 -> 20
- net +15V: track 640.7 -> 1114.6 mm, vias 9 -> 14
- net Net-(D18-Pad1): track 0.00 -> 332.3 mm
- net RECT15P: track 270.4 -> 0.00 mm
- net RECT15N: track 103.0 -> 0.00 mm
- net LEFTUNBAL: track 27.2 -> 119.5 mm
- net SUBUNBAL: track 0.00 -> 73.1 mm
- net POWERSW1: track 127.1 -> 186.1 mm
- net Net-(D5-Pad2): track 57.9 -> 11.9 mm
- net SUBMINUS: track 7.54 -> 48.0 mm
- net Net-(C59-Pad1): track 0.00 -> 40.1 mm
- net Net-(JP1-Pad1): track 61.9 -> 23.2 mm
- net RIGHTMINUS: track 9.09 -> 45.8 mm
- net Net-(D14-Pad2): track 0.00 -> 35.8 mm
- net Net-(D14-Pad1): track 35.8 -> 0.00 mm
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Other:
- board size 300 x 74 mm -> 300 x 90 mm
- board text added: "PRETTY GOOD PREAMPLIFIER V2 BY DANIEL MARKS CC-BY-SA 4.0"
- board text removed: "PRETTY GOOD PREAMPLIFIER BY DANIEL MARKS CC-BY-SA 4.0"

Commit message: JLCPCB order 2021-04-11
Parts:
- added C63: 100 nF, Capacitors_THT:C_Disc_D5.0mm_W2.5mm_P5.00mm, F.Cu at (207.2, 65.9)
- added JP3: PIN2, Pin_Headers:Pin_Header_Straight_1x02_Pitch2.54mm, F.Cu at (67.1, 53.1)
- added JP4: PIN2, Pin_Headers:Pin_Header_Straight_1x02_Pitch2.54mm, F.Cu at (67.1, 56.8)
- added R45: 100k, Resistors_THT:R_Axial_DIN0207_L6.3mm_D2.5mm_P7.62mm_Horizontal, F.Cu at (203.6, 69.5)
- added R46: 150R, Resistors_THT:R_Axial_DIN0309_L9.0mm_D3.2mm_P12.70mm_Horizontal, F.Cu at (67.0, 74.1)
- added R48: 100k, Resistors_THT:R_Axial_DIN0207_L6.3mm_D2.5mm_P7.62mm_Horizontal, F.Cu at (203.7, 72.7)
- C4, C5: value 1500 uF -> 2200 uF
- Q1: value 2N3906 -> 2N3904
- Q2: value TIP41C -> TIP42C
- R23: value 1k -> 3k3
- R42: value 10k -> 100k
- R43, R44: value 4R7 -> 1R
- moved D16 17.3 mm to (83.7, 75.4)
- moved JP2 13.1 mm to (162.5, 71.0), turned to 180 degrees
- moved R23 11.1 mm to (214.5, 81.1), turned to 90 degrees
- moved C49 8.04 mm to (120.7, 90.4)
- moved C50 7.92 mm to (111.5, 90.5)
- moved C3 7.49 mm to (120.7, 97.9)
- moved C7 7.39 mm to (115.7, 97.9)
- moved Q2 7.24 mm to (213.1, 56.5), turned to 270 degrees
- moved C55 2.36 mm to (184.8, 68.0)
- moved SW2 2.34 mm to (126.3, 67.0)
- moved SW3 2.32 mm to (77.9, 55.4)
- moved C57 2.30 mm to (189.8, 64.5)
- moved J17 1.92 mm to (197.5, 45.4)
- moved RLY9 1.81 mm to (314.3, 104.6)
- moved C53 1.70 mm to (120.7, 78.9)
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Connections:
- Q1 pad 1: +15V -> -15V
- Q1 pad 2: Net-(D17-Pad1) -> Net-(D17-Pad2)
- Q2 pad 3: GND -> +15V
- R23 pad 1: Net-(Q2-Pad1) -> Net-(Q1-Pad3)
- R23 pad 2: Net-(Q1-Pad3) -> Net-(Q2-Pad1)
Routing:
- net -15V: track 1149.7 -> 1292.6 mm, vias 20 -> 22
- net +15V: track 1114.6 -> 1248.7 mm
- net Net-(J24-Pad2): track 8.96 -> 34.5 mm
- net Net-(C63-Pad2): track 332.3 -> 356.7 mm
- net Net-(D17-Pad2): track 9.29 -> 26.5 mm
- net Net-(Q2-Pad1): track 8.73 -> 24.1 mm
- net Net-(J24-Pad1): track 19.7 -> 34.5 mm
- net Net-(C17-Pad1): track 105.9 -> 92.0 mm
- net Net-(D17-Pad1): track 18.2 -> 8.21 mm
- net Net-(C3-Pad1): track 41.7 -> 33.1 mm
- net Net-(C50-Pad1): track 3.45 -> 11.5 mm
- net Net-(C49-Pad1): track 3.50 -> 11.5 mm
- net Net-(C50-Pad2): track 40.8 -> 33.9 mm
- net Net-(C16-Pad2): track 104.0 -> 97.9 mm
- net Net-(JP4-Pad1): track 0.00 -> 4.64 mm
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Other:
- board text added: "LM317"
- board text added: "LM337"

Commit message: Moved around a component to make a little more space
Parts:
- removed JP3, JP4: PIN2, Pin_Headers:Pin_Header_Straight_1x02_Pitch2.54mm
- removed R46: 150R, Resistors_THT:R_Axial_DIN0309_L9.0mm_D3.2mm_P12.70mm_Horizontal
- added C64: 1500 uF, Capacitors_THT:CP_Radial_D10.0mm_P5.00mm, F.Cu at (67.0, 58.7)
- moved R1 17.3 mm to (74.5, 64.0), turned to 180 degrees
- moved C52 14.0 mm to (121.8, 88.5)
- moved C53 13.0 mm to (128.3, 89.5)
- moved D15 10.8 mm to (83.7, 70.3)
- moved C50 10.7 mm to (121.7, 93.6)
- moved D16 10.3 mm to (86.6, 85.3)
- moved C49 8.67 mm to (128.2, 94.7)
- moved C7 7.41 mm to (122.9, 99.7)
- moved C3 5.49 mm to (125.4, 100.8)
- moved C2 3.90 mm to (59.5, 77.5)
- moved D7 3.66 mm to (51.7, 102.2), turned to 270 degrees
- moved SW3 3.65 mm to (81.5, 54.9)
- moved C1 2.60 mm to (59.5, 95.2)
- moved RLY6 2.48 mm to (106.0, 66.9)
- moved J11 2.00 mm to (233.1, 45.7)
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Routing:
- net Net-(J24-Pad2): track 34.5 -> 7.80 mm
- net Net-(C64-Pad1): track 9.54 -> 34.8 mm
- net LEFTIN: track 17.9 -> 35.1 mm
- net Net-(J24-Pad1): track 34.5 -> 18.0 mm
- net RIGHTIN: track 14.5 -> 30.5 mm
- net Net-(C1-Pad1): track 34.3 -> 46.5 mm
- net Net-(C58-Pad2): track 42.2 -> 51.0 mm
- net Net-(J18-Pad2): track 33.0 -> 41.6 mm
- net Net-(RLY5-Pad2): track 25.3 -> 33.8 mm
- net Net-(C50-Pad2): track 33.9 -> 25.8 mm
- net Net-(C50-Pad1): track 11.5 -> 5.17 mm
- net -15V: track 1292.6 -> 1286.4 mm
- net Net-(C49-Pad1): track 11.5 -> 5.29 mm
- net +15V: track 1248.7 -> 1254.3 mm
- net Net-(JP4-Pad1): track 4.64 -> 0.00 mm
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
Commit message: Added jumpers to connect shields of XLR to ground
Parts:
- added C65: 1000 uF, Capacitors_THT:CP_Radial_D7.5mm_P2.50mm, F.Cu at (214.2, 63.7)
- added JP3: PH, Pin_Headers:Pin_Header_Straight_1x02_Pitch2.54mm, F.Cu at (28.9, 110.9)
- added JP4: PH, Pin_Headers:Pin_Header_Straight_1x02_Pitch2.54mm, F.Cu at (32.5, 110.9)
- added JP5: PH, Pin_Headers:Pin_Header_Straight_1x02_Pitch2.54mm, F.Cu at (314.7, 61.8)
- added JP6: PH, Pin_Headers:Pin_Header_Straight_1x02_Pitch2.54mm, F.Cu at (242.9, 59.0)
- added JP7: PH, Pin_Headers:Pin_Header_Straight_1x02_Pitch2.54mm, F.Cu at (282.8, 56.3)
- added JP8: PH, Pin_Headers:Pin_Header_Straight_1x02_Pitch2.54mm, F.Cu at (186.0, 55.4)
- added JP9: PH, Pin_Headers:Pin_Header_Straight_1x02_Pitch2.54mm, F.Cu at (159.4, 51.7)
- added L7: FB, Inductors_THT:L_Axial_L7.0mm_D3.3mm_P10.16mm_Horizontal_Fastron_MICC, F.Cu at (117.0, 85.8)
- added L8: FB, Inductors_THT:L_Axial_L7.0mm_D3.3mm_P10.16mm_Horizontal_Fastron_MICC, F.Cu at (127.2, 81.5)
- added R46: 10k, Resistors_THT:R_Axial_DIN0207_L6.3mm_D2.5mm_P7.62mm_Horizontal, F.Cu at (282.6, 94.8)
- C64: value 1500 uF -> 470 uF
- moved C2 47.5 mm to (104.1, 93.5), turned to 180 degrees
- moved R43 47.2 mm to (56.2, 93.8), turned to 270 degrees
- moved D16 39.9 mm to (63.3, 52.8), turned to 270 degrees
- moved C4 39.3 mm to (60.9, 88.1), turned to 90 degrees
- moved R44 32.7 mm to (71.5, 72.5)
- moved C59 30.4 mm to (73.2, 92.3), turned to 0 degrees
- moved R3 27.7 mm to (55.7, 112.9), turned to 270 degrees
- moved C58 26.4 mm to (59.4, 99.8), turned to 270 degrees
- moved R5 24.4 mm to (52.0, 112.8)
- moved SW3 20.0 mm to (98.3, 65.8)
- moved D15 18.7 mm to (82.3, 51.7), turned to 270 degrees
- moved D8 18.5 mm to (73.3, 89.1)
- moved R4 16.7 mm to (94.4, 83.4), turned to 270 degrees
- moved C5 13.2 mm to (80.0, 78.2), turned to 90 degrees
- moved R12 11.8 mm to (80.8, 119.8)
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Connections:
- C3 pad 1: Net-(C3-Pad1) -> GND
- C3 pad 2: GND -> Net-(C3-Pad2)
- C49 pad 1: Net-(C49-Pad1) -> Net-(C3-Pad2)
- C49 pad 2: Net-(C3-Pad1) -> Net-(C49-Pad2)
- C52 pad 1: Net-(C50-Pad1) -> Net-(C50-Pad2)
- C52 pad 2: LEFTIN -> Net-(C52-Pad2)
- C53 pad 1: Net-(C49-Pad1) -> Net-(C49-Pad2)
- C53 pad 2: RIGHTIN -> Net-(C53-Pad2)
- C7 pad 1: Net-(C50-Pad2) -> (no net)
- C7 pad 2: GND -> Net-(C52-Pad2)
- D11 pad 1: POWERSW2 -> Net-(D11-Pad1)
- J11 pad 1: GND -> Net-(J11-Pad1)
- J11 pad G: GND -> Net-(J11-Pad1)
- J12 pad 1: GND -> Net-(J12-Pad1)
- J12 pad G: GND -> Net-(J12-Pad1)
- J13 pad 1: GND -> Net-(J13-Pad1)
- J13 pad G: GND -> Net-(J13-Pad1)
- J16 pad 1: GND -> Net-(J16-Pad1)
- J16 pad G: GND -> Net-(J16-Pad1)
- J17 pad 1: GND -> Net-(J17-Pad1)
- J17 pad G: GND -> Net-(J17-Pad1)
- J3 pad 1: POWERSW1 -> Net-(J3-Pad1)
- J3 pad 2: POWERSW2 -> Net-(D11-Pad1)
- R1 pad 2: POWERSW1 -> Net-(J3-Pad1)
- R35 pad 2: Net-(C3-Pad1) -> Net-(C53-Pad2)
- R36 pad 1: Net-(C50-Pad2) -> Net-(C50-Pad1)
- RLY2 pad 5: POWERSW2 -> Net-(D11-Pad1)
- U6 pad 2: Net-(C31-Pad1) -> Net-(R46-Pad2)
Routing:
- net GND: track 0.00 -> 350.7 mm, vias 0 -> 101
- net POWERSW1: track 187.0 -> 105.1 mm
- net Net-(J3-Pad1): track 0.00 -> 79.9 mm
- net POWERSW2: track 161.0 -> 91.3 mm
- net Net-(D11-Pad1): track 0.00 -> 64.7 mm
- net +15V: track 1254.3 -> 1294.0 mm, vias 14 -> 15
- net Net-(C3-Pad1): track 30.4 -> 0.00 mm
- net Net-(C53-Pad2): track 0.00 -> 27.0 mm
- net Net-(C50-Pad2): track 25.8 -> 3.62 mm
- net Net-(J17-Pad1): track 0.00 -> 17.4 mm
- net Net-(J16-Pad1): track 0.00 -> 17.4 mm
- net Net-(C3-Pad2): track 0.00 -> 16.5 mm
- net Net-(J11-Pad1): track 0.00 -> 16.5 mm
- net Net-(C50-Pad1): track 5.17 -> 21.1 mm
- net RIGHTIN: track 30.5 -> 14.8 mm
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Other:
- board text added: "PRETTY GOOD PREAMPLIFIER V3 BY DANIEL MARKS CC-BY-SA 4.0"
- board text removed: "PRETTY GOOD PREAMPLIFIER V2 BY DANIEL MARKS CC-BY-SA 4.0"

Commit message: JLCPCB manufacturing
Parts:
- added C66: 47 uF, Capacitors_THT:CP_Radial_D5.0mm_P2.50mm, F.Cu at (313.1, 91.8)
- added C67: 47 uF, Capacitors_THT:CP_Radial_D5.0mm_P2.50mm, F.Cu at (318.9, 91.8)
- added C68: 47 uF, Capacitors_THT:CP_Radial_D5.0mm_P2.50mm, F.Cu at (267.6, 83.1)
- added C69: 47 uF, Capacitors_THT:CP_Radial_D5.0mm_P2.50mm, F.Cu at (267.6, 74.7)
- added C70: 47 uF, Capacitors_THT:CP_Radial_D5.0mm_P2.50mm, F.Cu at (221.2, 85.2)
- added C71: 47 uF, Capacitors_THT:CP_Radial_D5.0mm_P2.50mm, F.Cu at (215.6, 82.6)
- moved R31 23.9 mm to (312.9, 98.9), turned to 0 degrees
- moved R33 20.2 mm to (273.5, 71.4), turned to 180 degrees
- moved C1 11.5 mm to (61.6, 94.6)
- moved RLY8 10.1 mm to (318.7, 84.9)
- moved C63 8.71 mm to (202.6, 66.1), turned to 0 degrees
- moved R29 7.63 mm to (298.1, 82.9), turned to 0 degrees
- moved R30 7.58 mm to (272.5, 91.5), turned to 90 degrees
- moved U1 6.90 mm to (71.0, 109.5)
- moved C58 6.28 mm to (55.5, 104.7)
- moved R34 5.78 mm to (233.1, 85.4)
- moved R43 4.54 mm to (56.3, 89.2)
- moved C4 4.52 mm to (60.4, 83.6)
- moved R32 3.42 mm to (214.8, 88.0)
- moved C53 2.51 mm to (127.9, 99.6), turned to 90 degrees
- moved C52 2.51 mm to (122.1, 91.0), turned to 270 degrees
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Connections:
- C52 pad 1: Net-(C50-Pad2) -> Net-(C52-Pad1)
- C52 pad 2: Net-(C52-Pad2) -> Net-(C50-Pad2)
- C53 pad 1: Net-(C49-Pad2) -> Net-(C53-Pad1)
- C53 pad 2: Net-(C53-Pad2) -> Net-(C49-Pad2)
- C7 pad 1: (no net) -> Net-(C7-Pad1)
- C7 pad 2: Net-(C52-Pad2) -> Net-(C52-Pad1)
- J22 pad 3: (no net) -> Net-(J22-Pad3)
- L7 pad 1: Net-(C52-Pad2) -> Net-(C52-Pad1)
- R29 pad 1: SUBUNBAL -> Net-(C31-Pad1)
- R29 pad 2: Net-(C31-Pad1) -> Net-(C66-Pad1)
- R30 pad 1: LEFTUNBAL -> Net-(C39-Pad1)
- R30 pad 2: Net-(C39-Pad1) -> Net-(C68-Pad1)
- R32 pad 1: RIGHTUNBAL -> Net-(C70-Pad1)
- R35 pad 2: Net-(C53-Pad2) -> Net-(C53-Pad1)
- RLY1 pad 3: (no net) -> Net-(RLY1-Pad3)
- RLY1 pad 7: (no net) -> Net-(RLY1-Pad7)
- RLY10 pad 4: (no net) -> Net-(RLY10-Pad4)
- RLY10 pad 8: (no net) -> Net-(RLY10-Pad8)
- RLY11 pad 4: (no net) -> Net-(RLY11-Pad4)
- RLY11 pad 8: (no net) -> Net-(RLY11-Pad8)
- RLY12 pad 4: (no net) -> Net-(RLY12-Pad4)
- RLY12 pad 8: (no net) -> Net-(RLY12-Pad8)
- RLY2 pad 3: (no net) -> Net-(RLY2-Pad3)
- RLY2 pad 7: (no net) -> Net-(RLY2-Pad7)
- RLY7 pad 3: (no net) -> Net-(RLY7-Pad3)
- RLY7 pad 7: (no net) -> Net-(RLY7-Pad7)
- RLY8 pad 4: (no net) -> Net-(RLY8-Pad4)
- RLY8 pad 6: (no net) -> Net-(RLY8-Pad6)
- RLY8 pad 8: (no net) -> Net-(RLY8-Pad8)
- RLY9 pad 4: (no net) -> Net-(RLY9-Pad4)
- RLY9 pad 8: (no net) -> Net-(RLY9-Pad8)
Routing:
- net Net-(C53-Pad2): track 27.0 -> 0.00 mm
- net Net-(C53-Pad1): track 0.00 -> 27.0 mm
- net SUBUNBAL: track 72.0 -> 91.9 mm
- net Net-(C66-Pad1): track 0.00 -> 18.1 mm
- net LEFTUNBAL: track 122.4 -> 105.8 mm
- net RIGHTUNBAL: track 50.8 -> 65.6 mm
- net Net-(C52-Pad2): track 10.3 -> 0.00 mm
- net Net-(C52-Pad1): track 0.00 -> 10.3 mm
- net Net-(C70-Pad1): track 0.00 -> 7.60 mm
- net Net-(C70-Pad2): track 0.00 -> 6.61 mm
- net Net-(C58-Pad2): track 39.2 -> 33.2 mm
- net Net-(C39-Pad1): track 65.9 -> 71.8 mm
- net Net-(C66-Pad2): track 0.00 -> 5.84 mm
- net Net-(C68-Pad1): track 0.00 -> 5.67 mm
- net Net-(C63-Pad2): track 354.7 -> 349.1 mm
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
Commit message: A few minor changes to fix crowding of components
Parts:
- added C72: 22 pF, Capacitors_THT:C_Disc_D5.0mm_W2.5mm_P5.00mm, F.Cu at (271.9, 104.9)
- moved C33 11.8 mm to (280.8, 91.0), turned to 180 degrees
- moved C31 6.93 mm to (282.6, 99.9)
- moved C32 6.85 mm to (279.1, 99.9)
- moved R22 6.39 mm to (281.9, 115.1)
- moved R24 4.02 mm to (275.5, 105.5)
- moved R46 0.35 mm to (282.4, 94.6)
Routing:
- net -15V: track 1294.3 -> 1303.7 mm
- net Net-(R22-Pad1): track 26.1 -> 18.0 mm
- net Net-(C39-Pad1): track 71.8 -> 64.2 mm
- net Net-(C31-Pad2): track 39.7 -> 32.4 mm
- net Net-(C31-Pad1): track 51.0 -> 58.0 mm
- net Net-(R24-Pad1): track 23.0 -> 28.1 mm
- net +15V: track 1297.7 -> 1300.5 mm
- net Net-(C72-Pad2): track 9.05 -> 10.6 mm
- net Net-(C33-Pad2): track 19.0 -> 18.4 mm
